Commit message: [LIDAR] Add first lidar sensor to pybullet simulator

File: 006_simple_mobile_platform/simple_mobile_platform.xacro (robot description, xacro)
@@ -93,4 +93,27 @@
             </joint>
     </xacro:macro>
+<!-- ROBOT LIDAR -->
+    <xacro:macro name="lidar" params="name parent trans rot">
+        <link name="${name}">
+            <visual>
+                <geometry>
+                    <cylinder radius="0.02" length="0.05"/>
+                </geometry>
+            </visual>
+            <collision>
+                <geometry>
+                    <cylinder radius="0.02" length="0.05"/>
+                </geometry>
+            </collision>
+            <xacro:cylinder_inertia radius="0.3" length="0.2" mass="30">
+                <origin xyz="0 0 0" rpy="0 0 0"/>
+            </xacro:cylinder_inertia>
+        </link>
+        <joint name="${name}_joint" type="fixed">
+            <parent link="${parent}"/>
+            <child link="${name}"/>
+            <origin rpy="${rot}" xyz="${trans}"/>
+        </joint>
+    </xacro:macro>
 <!-- ASSEMBLY -->
     <link name="base_link"/>
@@ -99,4 +122,10 @@
         parent="base_link"
         trans="0 0 0"
+        rot="0 0 0"
+        />
+    <xacro:lidar
+        name="lidar"
+        parent="base_link"
+        trans="0.2 0 0.18"
         rot="0 0 0"
         />

Commit message: [LIDAR] Use pybullet querry instead of ros tf to find out position of lidar in world frame

File: 006_simple_mobile_platform/simple_mobile_platform.xacro (robot description, xacro)
@@ -117,8 +117,8 @@
     </xacro:macro>
 <!-- ASSEMBLY -->
-    <link name="base_link"/>
+    <link name="simple_mobile_platform"/>
     <xacro:frame
         name="frame"
-        parent="base_link"
+        parent="simple_mobile_platform"
         trans="0 0 0"
         rot="0 0 0"
@@ -126,5 +126,5 @@
     <xacro:lidar
         name="lidar"
-        parent="base_link"
+        parent="frame"
         trans="0.2 0 0.18"
         rot="0 0 0"
